File: AppleIIgsExpansionSlotBreakoutBoard.kicad_sch (KiCad schematic)
At the start: 5 parts, among them J1 Conn_02x25_Counter_Clockwise, J2 Conn_01x25, J3 Conn_01x25, J4 Conn_01x02, J5 Conn_01x02

Commit message: fixed DNA and INT lines not being connected.  cleaned up violations.
Other:
- note added: "DMA_OUT"
- note added: "INT_OUT"
Changed lines of the file:
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@@
+		)
+	)
+	(text "DMA_OUT"
+		(exclude_from_sim no)
+		(at 44.45 99.568 0)
+		(effects
+			(font
+				(size 1.27 1.27)
+			)
+		)
+	)
+	(text "INT_OUT"
+		(exclude_from_sim no)
+		(at 44.196 97.028 0)
+		(effects
+			(font
+				(size 1.27 1.27)
+			)
 		)
 	)
@@
 	)
 	(junction
-		(at 49.53 97.79)
-		(diameter 0)
-		(color 0 0 0 0)
-	)
-	(junction
-		(at 50.8 100.33)
-		(diameter 0)
-		(color 0 0 0 0)
-	)
-	(junction
 		(at 179.07 30.48)
 		(diameter 0)
@@
 	(wire
 		(pts
-			(xy 40.64 100.33) (xy 50.8 100.33)
-		)
-		(stroke
-			(width 0)
-			(type default)
-		)
-	)
-	(wire
-		(pts
 			(xy 40.64 64.77) (xy 52.07 64.77)
 		)
@@
 		(pts
 			(xy 50.8 100.33) (xy 50.8 105.41)
-		)
-		(stroke
-			(width 0)
-			(type default)
-		)
-	)
-	(wire
-		(pts
-			(xy 40.64 97.79) (xy 49.53 97.79)
 		)
 		(stroke
@@
 		)
 	)
-	(label "DMA_OUT"
-		(at 105.41 101.6 0)
+	(label "INT_IN"
+		(at 105.41 99.06 0)
 		(effects
 			(font
@@
 		)
 	)
-	(label "DMA_OUT"
-		(at 40.64 100.33 0)
-		(effects
-			(font
-				(size 1.27 1.27)
-			)
-			(justify left bottom)
-		)
-	)
 	(label "A3"
 		(at 105.41 53.34 0)
@@
 		)
 	)
-	(label "INT_OUT"
-		(at 105.41 99.06 0)
-		(effects
-			(font
-				(size 1.27 1.27)
-			)
-			(justify left bottom)
-		)
-	)
 	(label "~{IOSEL}"
 		(at 40.64 41.91 0)
@@
 		)
 	)
-	(label "INT_OUT"
-		(at 40.64 97.79 0)
-		(effects
-			(font
-				(size 1.27 1.27)
-			)
-			(justify left bottom)
-		)
-	)
 	(label "A2"
 		(at 105.41 50.8 0)
@@
 		(effects
 			(font
+				(size 1.27 1.27)
+			)
+			(justify left bottom)
+		)
+	)
+	(label "DMA_IN"
+		(at 105.41 101.6 0)
+		(effects
+			(font
